Commit message: Initial commit

File: linorobot2_description/urdf/2wd_properties.urdf.xacro (robot description, xacro)
@@ -1,19 +1,20 @@
 <?xml version="1.0"?>
 <robot xmlns:xacro="http://ros.org/wiki/xacro">
-  <xacro:property name="base_length" value="0.1435" />
-  <xacro:property name="base_width" value="0.1435" />
-  <xacro:property name="base_height" value="0.156" />
-  <xacro:property name="base_mass" value="1.2" />
-  <xacro:property name="wheel_radius" value="0.033" />
+  <xacro:property name="base_length" value="0.20" />
+  <xacro:property name="base_width" value="0.20" />
+  <xacro:property name="base_height" value="0.18852" />
+  <xacro:property name="base_mass" value="2.5" />
+  <xacro:property name="wheel_radius" value="0.0325" />
   <xacro:property name="wheel_width" value="0.027" />
   <xacro:property name="wheel_pos_x" value="0.0" />
-  <xacro:property name="wheel_pos_y" value="0.08675" />
-  <xacro:property name="wheel_pos_z" value="0.0238" />
-  <xacro:property name="wheel_mass" value="0.0334" />
+  <xacro:property name="wheel_pos_y" value="0.10688" />
+  <xacro:property name="wheel_pos_z" value="0.0325" />
+  <xacro:property name="wheel_mass" value="0.7181" />
   <xacro:property name="wheel_torque" value="0.43" />
   <xacro:property name="front_caster_wheel" value="false" />
-  <xacro:property name="rear_caster_wheel" value="true" />
+  <xacro:property name="rear_caster_wheel" value="false" />
+  <xacro:property name="wheel_coast" value="-0.0263800000000001" />
   <xacro:property name="laser_pose">
-    <origin xyz="-0.0331 0 0.208" rpy="0 0 0"/>
+    <origin xyz="0.00669528741938097 -7.83717636255732E-05 0.19525868699062" rpy="0 0 0"/>
   </xacro:property>
   <!-- Unused -->

File: linorobot2_description/urdf/controllers/diff_drive.urdf.xacro (robot description, xacro)
@@ -11,9 +11,9 @@
         <wheel_separation>${wheel_separation}</wheel_separation>
         <wheel_diameter>${wheel_radius * 2}</wheel_diameter>
-        <max_wheel_acceleration>1.0</max_wheel_acceleration>
+        <max_wheel_acceleration>40.0</max_wheel_acceleration>
         <robot_base_frame>base_footprint</robot_base_frame>
         <publish_odom>true</publish_odom>
         <publish_odom_tf>false</publish_odom_tf>
-        <publish_wheel_tf>true</publish_wheel_tf>
+        <publish_wheel_tf>true</publish_wheel_tf>  #da sua thanh true ---> false
         <odometry_frame>odom</odometry_frame>
       </plugin>

File: linorobot2_description/urdf/controllers/skid_steer.urdf.xacro (robot description, xacro)
@@ -17,5 +17,5 @@
         <updateRate>100</updateRate>
         <max_wheel_acceleration>1.0</max_wheel_acceleration>
-        <robot_base_frame>base_footprint</robot_base_frame>
+        <robot_base_frame>base_link</robot_base_frame>
         <publish_odom>true</publish_odom>
         <publish_odom_tf>false</publish_odom_tf>

File: linorobot2_description/urdf/mech/base.urdf.xacro (robot description, xacro)
@@ -2,12 +2,12 @@
 <robot xmlns:xacro="http://ros.org/wiki/xacro">
   <xacro:macro name="base" params="length width height mass wheel_radius wheel_pos_z">
-    <link name="base_footprint"/>
+    <link name="base_footprint" />
     <link name="base_link">
       <visual>
-        <origin xyz="-0.0276 0 0" rpy="0 0 0"/>
+        <origin xyz="0 0 0" rpy="0 0 0"/>
         <geometry>
           <!-- <box size="${length} ${width} ${height}"/> -->
           <!-- <mesh filename="" scale="0.001 0.001 0.001"/> -->
-          <mesh filename="package://linorobot2_description/meshes/lino_base.STL" scale="0.001 0.001 0.001"/>
+          <mesh filename="package://linorobot2_description/meshes/base_link.STL" scale="1 1 1"/>
         </geometry>
         <material name="light_black">
@@ -16,5 +16,6 @@
       </visual>
       <collision>
-        <origin xyz="-0.0276 0 ${height/2}" rpy="0 0 0"/>
+        <!-- <origin xyz="-0.0276 0 ${height/2}" rpy="0 0 0"/> -->
+        <origin xyz="0 0 ${height/2-wheel_pos_z}" rpy="0 0 0"/>
         <geometry>
           <box size="${length} ${width} ${height}"/>
@@ -22,10 +23,15 @@
       </collision>
       <inertial>
-        <origin xyz="-0.02957230 -0.00249250 0.04657955" rpy="0 0 0"/>
-        <mass value="${mass}"/>
-        <inertia ixx="0.00382227" ixy="-0.00007090" ixz="-0.00008756"
-                 iyy="0.00381152" iyz="-0.00003095"
-                 izz="0.00291391"/>
-      </inertial>
+      <origin
+        xyz="0 0 0" rpy="0 0 0" />
+      <mass value="2.5" />
+      <inertia
+        ixx="0.0116916235837784"
+        ixy="-8.10920537712205E-06"
+        ixz="3.2206377195194E-06"
+        iyy="0.010715791296685"
+        iyz="-2.38716537151557E-05"
+        izz="0.00946805534827865" />
+    </inertial>
     </link>
     <gazebo reference="base_link">
@@ -40,5 +46,5 @@
           <diffuse>0.4 0.4 0.4 1.0</diffuse>
           <specular>0.2 0.2 0.2 1.0</specular>
-          <emissive>0.0 0.0 0.0 0.0</emissive> -->
+          <emissive>0.0 0.0 0.0 0.0</emissive>   0.0342799999999999 -->
         </material>
       </visual>
@@ -48,5 +54,5 @@
       <parent link="base_footprint"/>
       <child link="base_link"/>
-      <origin xyz="0 0 0.0092" rpy="0 0 0"/>
+      <origin xyz="0 0 0.0325" rpy="0 0 0"/>
     </joint>
   </xacro:macro>

File: linorobot2_description/urdf/mech/caster_wheel.urdf.xacro (robot description, xacro)
@@ -2,16 +2,25 @@
 <robot xmlns:xacro="http://ros.org/wiki/xacro">
   <xacro:macro name="caster_wheel" params="side mass base_length wheel_radius wheel_pos_z">
-    <xacro:property name="caster_wheel_radius" value="0.0075" />
+    <!-- FRONT WHEEL CONFIG -->
     <xacro:if value="${side == 'front'}">
-        <xacro:property name="caster_wheel_x" value="${(base_length / 2) - caster_wheel_radius}" />
+      <xacro:property name="caster_wheel_radius" value="0.0325" />
+      <xacro:property name="caster_wheel_x" value="-0.0773955999155658" /> <!-- banh sau -->
+      <xacro:property name="caster_wheel_mass" value="1.7181" />
+      <xacro:property name="caster_mesh_file" value="front_caster_wheel.STL" />
+      <xacro:property name="caster_wheel_z" value="-0.026800000000001" />
     </xacro:if>
+    <!-- REAR WHEEL CONFIG -->
     <xacro:if value="${side == 'rear'}">
-        <xacro:property name="caster_wheel_x" value="-0.0661" />
+      <xacro:property name="caster_wheel_radius" value="0.0325" />
+      <xacro:property name="caster_wheel_x" value="0.0639497590100105" />
+      <xacro:property name="caster_wheel_mass" value="1.7191" />
+      <xacro:property name="caster_mesh_file" value="rear_caster_wheel.STL" />
+      <xacro:property name="caster_wheel_z" value="-0.026803000000001" />
     </xacro:if>
     <link name="${side}_caster_wheel_link">
       <visual>
-        <origin xyz="0 0 0" rpy="0 0 0"/>
+        <origin xyz="0 0 ${caster_wheel_z}" rpy="0 0 0"/>  <!-- ✅ Để ở (0,0,0) -->
         <geometry>
-          <sphere radius="${caster_wheel_radius}" />
+            <mesh filename="package://linorobot2_description/meshes/${caster_mesh_file}" scale="1 1 1"/>
         </geometry>
         <material name="white">
@@ -22,23 +31,23 @@
         <origin xyz="0 0 0" rpy="0 0 0"/>
         <geometry>
-          <sphere radius="${caster_wheel_radius}" />
+          <sphere radius="${caster_wheel_radius}"/>
         </geometry>
       </collision>
       <inertial>
         <origin xyz="0 0 0" rpy="0 0 0"/>
-        <mass value="${mass}"/>
-        <inertia ixx="${(2/5) * mass * (caster_wheel_radius * caster_wheel_radius)}" ixy="0" ixz="0"
-                 iyy="${(2/5) * mass * (caster_wheel_radius * caster_wheel_radius)}" iyz="0"
-                 izz="${(2/5) * mass * (caster_wheel_radius * caster_wheel_radius)}" />
+        <mass value="${caster_wheel_mass}"/>
+        <inertia ixx="${(2/5) * caster_wheel_mass * (caster_wheel_radius * caster_wheel_radius)}" ixy="0" ixz="0"
+                 iyy="${(2/5) * caster_wheel_mass * (caster_wheel_radius * caster_wheel_radius)}" iyz="0"
+                 izz="${(2/5) * caster_wheel_mass * (caster_wheel_radius * caster_wheel_radius)}" />
       </inertial>
     </link>
     <gazebo reference="${side}_caster_wheel_link">
-        <mu1>0.01</mu1>
-        <mu2>0.01</mu2>
+        <mu1>0.1</mu1>
+        <mu2>0.1</mu2>
     </gazebo>
     <joint name="${side}_caster_wheel_joint" type="fixed">
       <parent link="base_link"/>
       <child link="${side}_caster_wheel_link"/>
-      <origin xyz="${caster_wheel_x} 0 -0.002" rpy="0 0 0"/>
+      <origin xyz="${caster_wheel_x} 0 0" rpy="0 0 0"/>  <!-- ✅ Chỉ áp dụng ở joint -->
     </joint>
   </xacro:macro>

File: linorobot2_description/urdf/mech/wheel.urdf.xacro (robot description, xacro)
@@ -6,9 +6,9 @@
         <origin xyz="0 0 0" rpy="0 0 0"/>
         <geometry>
-          <!-- <cylinder radius="${radius}" length="${width}"/> -->
-          <mesh filename="package://linorobot2_description/meshes/wheel_${side}.STL" scale="0.001 0.001 0.001"/>
+        <!--  <cylinder radius="0.03578" length="${width}"/> -->
+           <mesh filename="package://linorobot2_description/meshes/wheel_${side}.STL" scale="1 1 1"/>
         </geometry>
         <material name="dark">
-          <color rgba="0.3 0.3 0.3 1.0"/>
+          <color rgba="0.9 0.5 0.3 1.0"/>
         </material>
       </visual>
@@ -22,6 +22,7 @@
         <origin xyz="0 0 0" rpy="0 0 0"/>
         <mass value="${mass}"/>
-        <inertia ixx="${(1/12) * mass * (3*radius*radius + width*width)}" ixy="0" ixz="0"
-                 iyy="${(1/2) * mass * (radius*radius)}" iyz="0"
+        <inertia ixx="${(1/12) * mass * (3*radius*radius + width*width)}" ixy="-8.10920537712205E-06"
+        ixz="3.2206377195194E-06"
+                 iyy="${(1/2) * mass * (radius*radius)}" iyz="-2.38716537151557E-05"
                  izz="${(1/12) * mass * (3*radius*radius + width*width)}" />
       </inertial>
@@ -44,5 +45,5 @@
     <joint name="${side}_wheel_joint" type="continuous">
       <axis xyz="0 1 0" />
-      <parent link="base_link"/>
+      <parent link="base_footprint"/>
       <child link="${side}_wheel_link"/>
       <origin xyz="${pos_x} ${pos_y} ${pos_z}" rpy="0 0 0"/>

File: linorobot2_description/urdf/robots/2wd.urdf.xacro (robot description, xacro)
@@ -18,4 +18,15 @@
     wheel_pos_z="${wheel_pos_z}"
 />
+<!--xyz=0.00004066, -0.10688, 0"  IGNORE   4.0661E-05 -0.10688 0 -->
+  <xacro:wheel
+    side="right"
+    radius="${wheel_radius}"
+    width="${wheel_width}"
+    pos_x="${wheel_pos_x}"
+    pos_y="${-wheel_pos_y}"
+    pos_z="${wheel_pos_z}"
+    mass="${wheel_mass}"
+  />
+<!---0.00001098, 0.10612, 0   -1.0982E-05 0.10612 0-->
   <xacro:wheel
     side="left"
@@ -27,13 +38,4 @@
     mass="${wheel_mass}"
   />
-  <xacro:wheel
-    side="right"
-    radius="${wheel_radius}"
-    width="${wheel_width}"
-    pos_x="${wheel_pos_x}"
-    pos_y="${-wheel_pos_y}"
-    pos_z="${wheel_pos_z}"
-    mass="${wheel_mass}"
-  />
   <xacro:if value="${front_caster_wheel}">
     <xacro:caster_wheel
@@ -42,5 +44,5 @@
       base_length="${base_length}"
       wheel_radius="${wheel_radius}"
-      wheel_pos_z="${wheel_pos_z}"
+      wheel_pos_z="-0.0263800000000001"
     />
   </xacro:if>
@@ -51,5 +53,5 @@
       base_length="${base_length}"
       wheel_radius="${wheel_radius}"
-      wheel_pos_z="${wheel_pos_z}"
+      wheel_pos_z="-0.0263800000000001"
     />
   </xacro:if>

File: linorobot2_description/urdf/sensors/imu.urdf.xacro (robot description, xacro)
@@ -5,5 +5,5 @@
       <parent link="base_link"/>
       <child link="imu_link"/>
-      <origin xyz="-0.07682 0 0.0826" rpy="0 0 0"/>
+      <origin xyz="0.07724 0.00013 0.04275" rpy="0 0 0"/>
     </joint>
     <gazebo reference="imu_link">

File: linorobot2_description/urdf/sensors/laser.urdf.xacro (robot description, xacro)
@@ -10,5 +10,5 @@
         <geometry>
           <!-- <cylinder radius="0.0375" length="0.05"/> -->
-          <mesh filename="package://linorobot2_description/meshes/lds.stl" scale="0.001 0.001 0.001"/>
+          <mesh filename="package://linorobot2_description/meshes/lidar.STL" scale="1 1 1"/>
         </geometry>
         <material name="dark">
@@ -17,5 +17,5 @@
       </visual>
       <collision>
-        <origin xyz="0.015 0 -0.015" rpy="0 0 0"/>
+        <origin xyz="0 0 0" rpy="0 0 0"/>
         <geometry>
           <cylinder radius="${ld_radius}" length="${ld_height}"/>
@@ -51,5 +51,5 @@
     </joint>
     <gazebo reference="${frame_id}">
-      <sensor type="gpu_ray" name="${frame_id}_lidar">
+      <sensor type="ray" name="${frame_id}_lidar"> #TODO: Change to "gpu_ray" for better performance, xoa gpu oi
         <always_on>true</always_on>
         <update_rate>${update_rate}</update_rate>
