Commit message: Cập nhật social_rl, perception, safety shield

File: linorobot2_description/urdf/2wd_properties.urdf.xacro (robot description, xacro)
@@ -18,8 +18,22 @@
     <origin xyz="0.00669528741938097 -7.83717636255732E-05 0.19525868699062" rpy="0 0 0"/>
   </xacro:property>
+  <!-- RGB-D camera carried by the robot, on the front edge of the base cover.
+       This is the only camera the social pipeline reads, so the three numbers
+       matter:
+         z = 0.2225 in base_link is 0.255 m above the ground, and it puts the
+             camera box (0.030 tall) entirely ABOVE the lidar plane at
+             z = 0.19526. Mounting it level with the lidar would make the
+             camera its own permanent obstacle in /scan.
+         x = 0.10  is the front edge of the 0.20 m base, clear of the lidar
+             body (radius 0.04).
+         pitch = -0.20 rad tilts it 11.5 deg UP. At 3 m the 87 x 70 deg frustum
+             then covers the ground up to 3.4 m high, i.e. two whole people; at
+             1.5 m it reaches 1.83 m, chest to neck. Closer than ~1.0 m their
+             heads leave the frame, which is what the VLM needs, so keep the
+             conversation pair at 1.5 m or more. -->
+  <xacro:property name="depth_sensor_pose">
+    <origin xyz="0.10 0.0 0.2225" rpy="0 -0.20 0"/>
+  </xacro:property>
   <!-- Unused -->
-  <xacro:property name="depth_sensor_pose">
-    <origin xyz="0.14 0.0 0.045" rpy="0 0 0"/>
-  </xacro:property>
   <xacro:property name="rear_camera_sensor_pose">
     <origin xyz="-0.14 0.0 0.045" rpy="0 0 3.14159"/>

File: linorobot2_description/urdf/robots/2wd.urdf.xacro (robot description, xacro)
@@ -7,5 +7,5 @@
   <xacro:include filename="$(find linorobot2_description)/urdf/sensors/imu.urdf.xacro" />
   <xacro:include filename="$(find linorobot2_description)/urdf/sensors/generic_laser.urdf.xacro" />
-  <!-- <xacro:include filename="$(find linorobot2_description)/urdf/sensors/depth_sensor.urdf.xacro" /> -->
+  <xacro:include filename="$(find linorobot2_description)/urdf/sensors/depth_sensor.urdf.xacro" />
   <!-- <xacro:include filename="$(find linorobot2_description)/urdf/sensors/camera.urdf.xacro" /> -->
   <xacro:include filename="$(find linorobot2_description)/urdf/controllers/diff_drive.urdf.xacro" />
@@ -60,7 +60,7 @@
     <xacro:insert_block name="laser_pose" />
   </xacro:generic_laser>
-  <!-- <xacro:depth_sensor>
+  <xacro:depth_sensor>
     <xacro:insert_block name="depth_sensor_pose" />
-  </xacro:depth_sensor> -->
+  </xacro:depth_sensor>
   <!-- <xacro:rgb_camera
       parent="base_link"

File: linorobot2_description/urdf/sensors/depth_sensor.urdf.xacro (robot description, xacro)
@@ -52,5 +52,11 @@
       <sensor name="camera" type="depth">
         <always_on>true</always_on>
-        <update_rate>30.0</update_rate>
+        <!-- Rendering RGB *and* depth at 640x480 is the steadiest CPU load in
+             the whole sim, and the VLM worker is serial at one inference per
+             ~2 s (vlm_inference_interval), so frames past ~8 Hz are rendered
+             only to be dropped. YOLO tracking still updates every frame.
+             maximum_depth_age in social_vlm_perception.yaml is scaled to this
+             rate, so raise both together or neither. -->
+        <update_rate>8.0</update_rate>
         <camera name="camera">
           <horizontal_fov>1.50098</horizontal_fov>
@@ -60,4 +66,10 @@
             <format>R8G8B8</format>
           </image>
+          <!-- People are tracked out to maximum_depth = 12.0 m. The default
+               far plane would render scenery no one measures. -->
+          <clip>
+            <near>0.1</near>
+            <far>12.0</far>
+          </clip>
         </camera>
         <plugin name="depth_camera_controller" filename="libgazebo_ros_camera.so">
@@ -76,5 +88,8 @@
           </ros>
           <min_depth>0.015</min_depth>
-          <max_depth>3.0</max_depth>
+          <!-- Was 3.0, which clamped every person past 3 m to the same reading
+               and made them unusable to the tracker. Matches maximum_depth in
+               social_vlm_perception.yaml. -->
+          <max_depth>12.0</max_depth>
           <hack_baseline>0.07</hack_baseline>
           <frame_name>camera_depth_link</frame_name>
