Commit message: Update social navigation

File: linorobot2_description/urdf/controllers/diff_drive.urdf.xacro (robot description, xacro)
@@ -5,4 +5,5 @@
         <ros>
           <remapping>odom:=odom/unfiltered</remapping>
+          <remapping>cmd_vel:=cmd_vel_safe</remapping>
         </ros>
         <updateRate>100</updateRate>

File: linorobot2_description/urdf/controllers/skid_steer.urdf.xacro (robot description, xacro)
@@ -5,4 +5,5 @@
         <ros>
           <remapping>odom:=odom/unfiltered</remapping>
+          <remapping>cmd_vel:=cmd_vel_safe</remapping>
         </ros>
         <num_wheel_pairs>2</num_wheel_pairs>

File: linorobot2_description/urdf/mech/base.urdf.xacro (robot description, xacro)
@@ -9,5 +9,5 @@
           <!-- <box size="${length} ${width} ${height}"/> -->
           <!-- <mesh filename="" scale="0.001 0.001 0.001"/> -->
-          <mesh filename="package://linorobot2_description/meshes/base_link.STL" scale="1 1 1"/>
+          <mesh filename="file://$(find linorobot2_description)/meshes/base_link.STL" scale="1 1 1"/>
         </geometry>
         <material name="light_black">

File: linorobot2_description/urdf/mech/caster_wheel.urdf.xacro (robot description, xacro)
@@ -22,5 +22,5 @@
         <origin xyz="0 0 ${caster_wheel_z}" rpy="0 0 0"/>  <!-- ✅ Để ở (0,0,0) -->
         <geometry>
-            <mesh filename="package://linorobot2_description/meshes/${caster_mesh_file}" scale="1 1 1"/>
+            <mesh filename="file://$(find linorobot2_description)/meshes/${caster_mesh_file}" scale="1 1 1"/>
         </geometry>
         <material name="white">

File: linorobot2_description/urdf/mech/wheel.urdf.xacro (robot description, xacro)
@@ -7,5 +7,5 @@
         <geometry>
         <!--  <cylinder radius="0.03578" length="${width}"/> -->
-           <mesh filename="package://linorobot2_description/meshes/wheel_${side}.STL" scale="1 1 1"/>
+           <mesh filename="file://$(find linorobot2_description)/meshes/wheel_${side}.STL" scale="1 1 1"/>
         </geometry>
         <material name="dark">

File: linorobot2_description/urdf/sensors/laser.urdf.xacro (robot description, xacro)
@@ -10,5 +10,5 @@
         <geometry>
           <!-- <cylinder radius="0.0375" length="0.05"/> -->
-          <mesh filename="package://linorobot2_description/meshes/lidar.STL" scale="1 1 1"/>
+          <mesh filename="file://$(find linorobot2_description)/meshes/lidar.STL" scale="1 1 1"/>
         </geometry>
         <material name="dark">

Commit message: first commit

File: linorobot2_description/urdf/controllers/diff_drive.urdf.xacro (robot description, xacro)
@@ -15,6 +15,14 @@
         <robot_base_frame>base_footprint</robot_base_frame>
         <publish_odom>true</publish_odom>
+        <!-- False on purpose: odometry goes out on /odom/unfiltered and the
+             EKF in gazebo.launch.py is what fuses it and publishes
+             odom -> base_footprint. Launching with run_ekf:=false therefore
+             leaves nothing publishing that transform, the `odom` frame never
+             comes into existence, and Nav2 cannot start: local_costmap times
+             out on base_link -> odom and AMCL drops every scan. Set this to
+             true only if you also intend to run without the EKF. -->
         <publish_odom_tf>false</publish_odom_tf>
-        <publish_wheel_tf>true</publish_wheel_tf>  #da sua thanh true ---> false
+        <!-- ghi chú cũ giữ lại: "da sua thanh true, roi doi thanh false" -->
+        <publish_wheel_tf>true</publish_wheel_tf>
         <odometry_frame>odom</odometry_frame>
       </plugin>

File: linorobot2_description/urdf/mech/base.urdf.xacro (robot description, xacro)
@@ -9,5 +9,5 @@
           <!-- <box size="${length} ${width} ${height}"/> -->
           <!-- <mesh filename="" scale="0.001 0.001 0.001"/> -->
-          <mesh filename="file://$(find linorobot2_description)/meshes/base_link.STL" scale="1 1 1"/>
+          <mesh filename="package://linorobot2_description/meshes/base_link.STL" scale="1 1 1"/>
         </geometry>
         <material name="light_black">

File: linorobot2_description/urdf/mech/caster_wheel.urdf.xacro (robot description, xacro)
@@ -22,5 +22,5 @@
         <origin xyz="0 0 ${caster_wheel_z}" rpy="0 0 0"/>  <!-- ✅ Để ở (0,0,0) -->
         <geometry>
-            <mesh filename="file://$(find linorobot2_description)/meshes/${caster_mesh_file}" scale="1 1 1"/>
+            <mesh filename="package://linorobot2_description/meshes/${caster_mesh_file}" scale="1 1 1"/>
         </geometry>
         <material name="white">

File: linorobot2_description/urdf/mech/wheel.urdf.xacro (robot description, xacro)
@@ -7,5 +7,5 @@
         <geometry>
         <!--  <cylinder radius="0.03578" length="${width}"/> -->
-           <mesh filename="file://$(find linorobot2_description)/meshes/wheel_${side}.STL" scale="1 1 1"/>
+           <mesh filename="package://linorobot2_description/meshes/wheel_${side}.STL" scale="1 1 1"/>
         </geometry>
         <material name="dark">

File: linorobot2_description/urdf/sensors/depth_sensor.urdf.xacro (robot description, xacro)
@@ -36,5 +36,5 @@
         </material>
       </visual>
-    </gazebo>rgb(213,28,40)
+    </gazebo>
     <joint name="camera_to_base_link" type="fixed">
       <parent link="base_link"/>

File: linorobot2_description/urdf/sensors/laser.urdf.xacro (robot description, xacro)
@@ -10,5 +10,5 @@
         <geometry>
           <!-- <cylinder radius="0.0375" length="0.05"/> -->
-          <mesh filename="file://$(find linorobot2_description)/meshes/lidar.STL" scale="1 1 1"/>
+          <mesh filename="package://linorobot2_description/meshes/lidar.STL" scale="1 1 1"/>
         </geometry>
         <material name="dark">
@@ -51,5 +51,6 @@
     </joint>
     <gazebo reference="${frame_id}">
-      <sensor type="ray" name="${frame_id}_lidar"> #TODO: Change to "gpu_ray" for better performance, xoa gpu oi
+      <!-- TODO: change to "gpu_ray" for better performance -->
+      <sensor type="ray" name="${frame_id}_lidar">
         <always_on>true</always_on>
         <update_rate>${update_rate}</update_rate>
